File: ProjectBoard/Drummer_Project.brd (EAGLE design)
At the start: 71.1 x 37.5 mm, 9 parts, among them J1 292303-1, SW1 PUSH_BUTTON, U1 POCKETBEAGLE, U2 SERVO_SG90, U3 SERVO_SG90

Commit message: Changes!
here
Connections:
- removed net N$23: SW1.1, SW1.3, U1.P1_01, U1.P1_02, U1.P1_07, U1.P1_14, U1.P1_17, U1.P1_18, U1.P1_19, U1.P1_21, U1.P1_23, U1.P1_25, U1.P1_27, U1.P2_12, U1.P2_13, U1.P2_14, U1.P2_16, U1.P2_23, U1.P2_24, U1.P2_26, U1.P2_36, U2.PWR, U3.PWR
- removed net VDD_3P3V: U1.P1_24
- new net N$1: SW1.3, U1.P2_24
- new net VDD_3V3: SW1.1, U1.P1_01, U1.P1_02, U1.P1_07, U1.P1_14, U1.P1_17, U1.P1_18, U1.P1_19, U1.P1_21, U1.P1_23, U1.P1_24, U1.P1_25, U1.P1_27, U1.P2_12, U1.P2_13, U1.P2_14, U1.P2_16, U1.P2_23, U1.P2_26, U1.P2_36, U2.PWR, U3.PWR
Routing:
- net N$1: track 0.00 -> 20.0 mm
- net N$23: track 18.1 -> 0.00 mm
- added copper zone on layer 16, net VDD_3V3
- removed copper zone on layer 16, net N$23
Changed lines of the file:
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@@
 <layer number="56" name="wert" color="7" fill="1" visible="no" active="no"/>
 <layer number="57" name="tCAD" color="7" fill="1" visible="no" active="no"/>
+<layer number="58" name="tCAD" color="7" fill="1" visible="no" active="no"/>
 <layer number="59" name="tCarbon" color="7" fill="1" visible="no" active="no"/>
 <layer number="60" name="bCarbon" color="7" fill="1" visible="no" active="no"/>
@@
 <wire x1="18.229" y1="7.81345" x2="18.229" y2="6.197" width="0.254" layer="1"/>
 </signal>
-<signal name="N$23">
+<signal name="VDD_3V3">
 <contactref element="U2" pad="PWR"/>
 <contactref element="U3" pad="PWR"/>
 <contactref element="U1" pad="P1_14"/>
-<contactref element="SW1" pad="1"/>
-<contactref element="U1" pad="P2_24"/>
-<contactref element="SW1" pad="3"/>
 <contactref element="U1" pad="P1_01"/>
 <contactref element="U1" pad="P2_13"/>
@@
 <vertex x="76.2" y="43.18"/>
 </polygon>
-<wire x1="38.762" y1="16.296" x2="34.866" y2="20.192" width="0.254" layer="16"/>
-<wire x1="34.866" y1="20.192" x2="34.866" y2="32.74" width="0.254" layer="16"/>
-</signal>
-<signal name="VDD_3P3V">
+<contactref element="SW1" pad="1"/>
 <contactref element="U1" pad="P1_24"/>
 </signal>
+<signal name="N$1">
+<contactref element="SW1" pad="3"/>
+<contactref element="U1" pad="P2_24"/>
+<wire x1="34.866" y1="31.81645" x2="34.866" y2="32.74" width="0.254" layer="16"/>
+<wire x1="33.723" y1="30.67345" x2="34.866" y2="31.81645" width="0.254" layer="16"/>
+<wire x1="26.262" y1="16.296" x2="33.723" y2="23.757" width="0.254" layer="16"/>
+<wire x1="33.723" y1="23.757" x2="33.723" y2="30.67345" width="0.254" layer="16"/>
+</signal>
 </signals>
